File: hardware/relay-board-revC/relay_board.kicad_sch (KiCad schematic)
At the start: 144 parts, among them J1 USB-C, J10 DUT A F, J11 DUT A S, J12 DUT B F, J13 DUT B S, J14 DUT C F, J15 DUT C S, J16 DUT D F, J17 DUT D S, J6 BNC SOURCE, J7 BNC CH1, J8 SWD, J9 BNC CH2, K1 G6K-2F-RF-S DC5, K10 G6K-2F-RF-S DC5, K11 G6K-2F-RF-S DC5, K12 G6K-2F-RF-S DC5, K13 G6K-2F-RF-S DC5, K14 G6K-2F-RF-S DC5, K15 G6K-2F-RF-S DC5, K16 G6K-2F-RF-S DC5, K17 G6K-2F-RF-S DC5, K18 G6K-2F-RF-S DC5, K19 G6K-2F-RF-S DC5, K2 G6K-2F-RF-S DC5, K20 G6K-2F-RF-S DC5, K21 G6K-2F-RF-S DC5, K22 G6K-2F-RF-S DC5, K23 G6K-2F-RF-S DC5, K3 G6K-2F-RF-S DC5, K4 G6K-2F-RF-S DC5, K5 G6K-2F-RF-S DC5, K6 G6K-2F-RF-S DC5, K7 G6K-2F-RF-S DC5, K8 G6K-2F-RF-S DC5, K9 G6K-2F-RF-S DC5, SW1 BOOT, SW2 RESET, U1 STM32F072CBT6, U10 OPA356, U11 TPS2051CDBV, U12 TMP117AIDRV, U2 TBD62003APG, U3 TBD62003APG, U4 TBD62003APG, U5 AP2112K-3.3, U6 TBD62003APG, U7 OPA356, U8 OPA356, U9 OPA356

Commit message: Rev C as built: design, fab and JLC files of the manufactured boards
Schematic, routed PCB, netlist, generator/router scripts and docs as sent
to JLCPCB (fab outputs of 2026-10-13), Grayhill 02-21 clip footprint, the
via-out-of-pad fixes, the driven-guard study, BOM, JLC BOM/CPL, the fab
bundle and the review zip for N. Rosano. relay_map_revc.h is the map
generated from this schematic, checked against the netlist and flashed on
both built boards (firmware 2.0.0).

Co-Authored-By: Claude Opus 5.5 <noreply@anthropic.com>
Parts:
- added C37: 100nF, Capacitor_SMD:C_0402_1005Metric, symbol Device:C
- J10, J11, J12, J13, J14, J15, J16, J17: footprint Connector:Banana_Jack_1Pin -> OpenMagnetics:Grayhill_02-21_BananaPlug_4mm
Connections:
- net +5V_IN: now also C37.1
- net GND: now also C37.2
- net GPIO15: now also U1.12 (PA2); no longer U1.10 (PA0)
- net GPIO16: now also U1.5 (PF0); no longer U1.6 (PF1)
- net GPIO17: now also U1.4 (PC15); no longer U1.5 (PF0)
- net GPIO18: now also U1.3 (PC14); no longer U1.4 (PC15)
- net GPIO19: now also U1.2 (PC13); no longer U1.3 (PC14)
- net GPIO22: now also U1.10 (PA0); no longer U1.12 (PA2)
